File: JackFxTx.kicad_pcb (KiCad board)
At the start: 2 copper layers, 38 parts, among them J1 NRJ6HM-1, J2 USB_C_Receptacle_USB2.0_14P, SW1 SW_Push, SW2 SW_Push, SW3 SW_SPDT, U1 ESP32-S3-WROOM-1, U2 MCP6001-OT, U3 MCP73831-2-OT, U4 PCM1860DBT, U5 AP2112K-3.3, Y1 25 MHz

Commit message: update
Parts:
- added C20: 10 µF, Capacitor_SMD:C_0805_2012Metric_Pad1.18x1.45mm_HandSolder, F.Cu at (183.9, 98.6)
- added C21: 100 nF, Capacitor_SMD:C_0805_2012Metric_Pad1.18x1.45mm_HandSolder, F.Cu at (183.9, 101.6)
- added C22: 10 µF, Capacitor_SMD:C_0805_2012Metric_Pad1.18x1.45mm_HandSolder, F.Cu at (183.9, 104.6)
- R3: value 2 kR -> 4.7 kR
- moved Y1 66.9 mm to (176.4, 72.0)
- moved SW3 51.7 mm to (122.0, 134.1)
- moved C2 48.8 mm to (169.5, 98.6)
- moved C3 48.8 mm to (169.5, 101.6)
- moved C5 48.8 mm to (169.5, 107.6)
- moved C6 48.8 mm to (169.5, 110.7)
- moved C1 48.8 mm to (169.5, 95.6)
- moved C4 48.8 mm to (169.5, 104.6)
- moved C10 48.8 mm to (174.3, 104.6)
- moved C11 48.8 mm to (174.3, 107.6)
- moved C12 48.8 mm to (174.3, 110.7)
- moved C13 48.8 mm to (179.1, 95.6)
- moved C14 48.8 mm to (179.1, 98.6)
- moved C15 48.8 mm to (179.1, 101.6)
- moved C7 48.8 mm to (174.3, 95.6)
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Connections:
- U4 pad 15: unconnected-(U4-SCKI-Pad15) -> GND
