File: JackFxTx.kicad_sch (KiCad schematic)
At the start: 38 parts, among them J1 NRJ6HM-1, J2 USB_C_Receptacle_USB2.0_14P, SW1 SW_Push, SW2 SW_Push, SW3 SW_SPDT, U1 ESP32-S3-WROOM-1, U2 MCP6001-OT, U3 MCP73831-2-OT, U4 PCM1860DBT, U5 AP2112K-3.3, Y1 25 MHz

Commit message: update
Parts:
- added C20, C22: 10 µF, Capacitor_SMD:C_0805_2012Metric_Pad1.18x1.45mm_HandSolder, symbol Device:C
- added C21: 100 nF, Capacitor_SMD:C_0805_2012Metric_Pad1.18x1.45mm_HandSolder, symbol Device:C
- R3: value 2 kR -> 4.7 kR
Connections:
- net +3.3V: now also C22.1
- net GND: now also U4.15 (SCKI), C20.1, C21.1, C22.2
- net at C6.2, SW3.2 (B), U5.1 (VIN)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: now also C20.2, C21.2
- no-connect marks 39 -> 38
Other:
- moved on the sheet: C15, C2, C6, R1, R3, SW1, SW2, SW3, U1, U3, U5
